File: CZTBoardV3/CZTBoardV3.brd (EAGLE design)
At the start: 80 x 100.1 mm, 37 parts, among them IC1 LD117AS33TR, IC2 LD117AS33TR, X6 GX16

Commit message: Updated to final design and created output paths
Parts:
- moved X6 0.25 mm to (30.5, 91.4)
Routing:
- net GND: vias 1 -> 5
Other:
- board size 80 x 100.1 mm -> 80 x 100 mm
- board text removed: "CZT INTERFACE CARD V3 - TOP"
Changed lines of the file:
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@@
 <grid distance="10" unitdist="mil" unit="mm" style="lines" multiple="1" display="yes" altdistance="1" altunitdist="mm" altunit="mm"/>
 <layers>
-<layer number="1" name="Top" color="4" fill="1" visible="no" active="yes"/>
+<layer number="1" name="Top" color="4" fill="1" visible="yes" active="yes"/>
 <layer number="16" name="Bottom" color="1" fill="1" visible="yes" active="yes"/>
 <layer number="17" name="Pads" color="2" fill="1" visible="yes" active="yes"/>
@@
 <layer number="19" name="Unrouted" color="6" fill="1" visible="no" active="yes"/>
 <layer number="20" name="Dimension" color="24" fill="1" visible="yes" active="yes"/>
-<layer number="21" name="tPlace" color="7" fill="1" visible="no" active="yes"/>
-<layer number="22" name="bPlace" color="7" fill="1" visible="no" active="yes"/>
-<layer number="23" name="tOrigins" color="15" fill="1" visible="no" active="yes"/>
-<layer number="24" name="bOrigins" color="15" fill="1" visible="no" active="yes"/>
-<layer number="25" name="tNames" color="7" fill="1" visible="no" active="yes"/>
-<layer number="26" name="bNames" color="7" fill="1" visible="no" active="yes"/>
-<layer number="27" name="tValues" color="7" fill="1" visible="no" active="yes"/>
-<layer number="28" name="bValues" color="7" fill="1" visible="no" active="yes"/>
+<layer number="21" name="tPlace" color="7" fill="1" visible="yes" active="yes"/>
+<layer number="22" name="bPlace" color="7" fill="1" visible="yes" active="yes"/>
+<layer number="23" name="tOrigins" color="15" fill="1" visible="yes" active="yes"/>
+<layer number="24" name="bOrigins" color="15" fill="1" visible="yes" active="yes"/>
+<layer number="25" name="tNames" color="7" fill="1" visible="yes" active="yes"/>
+<layer number="26" name="bNames" color="7" fill="1" visible="yes" active="yes"/>
+<layer number="27" name="tValues" color="7" fill="1" visible="yes" active="yes"/>
+<layer number="28" name="bValues" color="7" fill="1" visible="yes" active="yes"/>
 <layer number="29" name="tStop" color="7" fill="3" visible="no" active="yes"/>
 <layer number="30" name="bStop" color="7" fill="6" visible="no" active="yes"/>
@@
 <layer number="44" name="Drills" color="7" fill="1" visible="no" active="yes"/>
 <layer number="45" name="Holes" color="7" fill="1" visible="yes" active="yes"/>
-<layer number="46" name="Milling" color="3" fill="1" visible="no" active="yes"/>
+<layer number="46" name="Milling" color="3" fill="1" visible="yes" active="yes"/>
 <layer number="47" name="Measures" color="7" fill="1" visible="no" active="yes"/>
 <layer number="48" name="Document" color="7" fill="1" visible="no" active="yes"/>
@@
 <wire x1="80" y1="0" x2="80" y2="100" width="0" layer="20"/>
 <wire x1="80" y1="100" x2="0" y2="100" width="0" layer="20"/>
-<wire x1="0" y1="100" x2="0" y2="88.138" width="0" layer="20"/>
-<text x="54.61" y="73.152" size="1.778" layer="1" font="vector">CZT INTERFACE
-CARD V3 - TOP</text>
 <text x="71.12" y="65.786" size="1.778" layer="16" font="vector" rot="MR0">MAR 2021
 ~HSB</text>
-<wire x1="0" y1="83" x2="0" y2="0" width="0" layer="20"/>
-<wire x1="0" y1="83" x2="0" y2="88.138" width="0.1524" layer="20"/>
-<wire x1="0" y1="88.138" x2="0" y2="100.076" width="0.1524" layer="20"/>
-<wire x1="0" y1="100.076" x2="80.01" y2="100.076" width="0.1524" layer="20"/>
-<wire x1="80.01" y1="100.076" x2="80.01" y2="83" width="0.1524" layer="20"/>
-<wire x1="80.01" y1="83" x2="0" y2="83" width="0.1524" layer="20"/>
-<wire x1="0.254" y1="94.742" x2="7.112" y2="94.742" width="0.1524" layer="20"/>
-<wire x1="0.254" y1="88.138" x2="7.112" y2="88.138" width="0.1524" layer="20"/>
-<wire x1="7.112" y1="94.742" x2="7.112" y2="99.568" width="0.1524" layer="20"/>
-<wire x1="7.112" y1="88.138" x2="7.112" y2="83.312" width="0.1524" layer="20"/>
-<wire x1="73.152" y1="88.138" x2="73.152" y2="83.312" width="0.1524" layer="20"/>
-<wire x1="72.898" y1="94.742" x2="72.898" y2="99.568" width="0.1524" layer="20"/>
-<wire x1="72.898" y1="94.742" x2="79.756" y2="94.742" width="0.1524" layer="20"/>
-<wire x1="73.152" y1="88.138" x2="79.756" y2="88.138" width="0.1524" layer="20"/>
+<wire x1="0" y1="100" x2="0" y2="0" width="0" layer="20"/>
+<polygon width="0.1524" layer="46" pour="hatch">
+<vertex x="13.716" y="64.262"/>
+<vertex x="13.716" y="53.086"/>
+<vertex x="20.828" y="53.086"/>
+<vertex x="20.828" y="64.262"/>
+</polygon>
+<polygon width="0.1524" layer="46">
+<vertex x="45.974" y="96.52"/>
+<vertex x="45.974" y="86.52"/>
+<vertex x="65.974" y="86.52"/>
+<vertex x="65.974" y="96.52"/>
+</polygon>
+<dimension x1="0" y1="100.076" x2="0" y2="0" x3="-13.716" y3="50.038" textsize="1.778" layer="20" dtype="vertical"/>
+<dimension x1="0" y1="0" x2="80.01" y2="1.27" x3="40.005" y3="-8.636" textsize="1.778" layer="20" dtype="horizontal"/>
+<dimension x1="0" y1="80.01" x2="0" y2="0" x3="-5.842" y3="40.005" textsize="1.778" layer="20"/>
 </plain>
 <attributes>
@@
 <element name="C2" library="rcl" package="C0805K" value="0.1u" x="48.768" y="34.544" smashed="yes" rot="R180">
 <attribute name="NAME" x="49.768" y="36.463" size="1.016" layer="25" rot="R180"/>
-<attribute name="VALUE" x="49.768" y="36.444" size="1.016" layer="27" rot="R180"/>
+<attribute name="VALUE" x="46.72" y="35.174" size="1.016" layer="27" rot="R180"/>
 </element>
 <element name="C3" library="rcl" package="C0805K" value="0.01u" x="63.754" y="42.418" smashed="yes" rot="R180">
 <attribute name="NAME" x="64.754" y="41.543" size="1.016" layer="25" rot="R180"/>
-<attribute name="VALUE" x="64.754" y="44.318" size="1.016" layer="27" rot="R180"/>
+<attribute name="VALUE" x="65.262" y="44.572" size="1.016" layer="27" rot="R180"/>
 </element>
 <element name="C4" library="rcl" package="C0805K" value="0.001u" x="31.496" y="36.068" smashed="yes">
@@
 </element>
 <element name="R1" library="rcl" package="R1206" value="100" x="41.402" y="30.734" smashed="yes" rot="R180">
-<attribute name="NAME" x="42.418" y="33.274" size="1.27" layer="25" rot="R180"/>
+<attribute name="NAME" x="38.608" y="31.242" size="1.27" layer="25" rot="R180"/>
 <attribute name="VALUE" x="42.672" y="33.274" size="1.27" layer="27" rot="R180"/>
 </element>
 <element name="R11" library="rcl" package="R1206" value="10k" x="14.478" y="11.938" smashed="yes" rot="R180">
 <attribute name="NAME" x="14.986" y="14.224" size="1.27" layer="25" rot="R180"/>
-<attribute name="VALUE" x="15.748" y="14.478" size="1.27" layer="27" rot="R180"/>
+<attribute name="VALUE" x="11.684" y="14.224" size="1.27" layer="27" rot="R180"/>
 </element>
 <element name="R12" library="rcl" package="R1206" value="10k" x="69.596" y="23.368" smashed="yes" rot="R180">
@@
 <element name="R7" library="rcl" package="R1206" value="0" x="36.068" y="18.034" smashed="yes">
 <attribute name="NAME" x="34.798" y="19.304" size="1.27" layer="25"/>
-<attribute name="VALUE" x="34.798" y="15.494" size="1.27" layer="27"/>
+<attribute name="VALUE" x="33.528" y="19.304" size="1.27" layer="27"/>
 </element>
 <element name="R8" library="rcl" package="R1206" value="0" x="16.002" y="18.542" smashed="yes" rot="R90">
 <attribute name="NAME" x="14.732" y="17.272" size="1.27" layer="25" rot="R90"/>
-<attribute name="VALUE" x="18.542" y="17.272" size="1.27" layer="27" rot="R90"/>
+<attribute name="VALUE" x="12.954" y="18.542" size="1.27" layer="27" rot="R90"/>
 </element>
 <element name="U$1" library="Orbotech_OMS40G256" package="ORBOTECH_OMS40G256" value="ORBOTECH_OMS40G256" x="1.778" y="78.232" locked="yes" smashed="yes" rot="R270">
@@
 <attribute name="VALUE" x="9.906" y="84.074" size="1.778" layer="27"/>
 </element>
-<element name="X6" library="TI_Downloaded" package="GX16" value="GX16" x="30.226" y="91.44" smashed="yes"/>
+<element name="X6" library="TI_Downloaded" package="GX16" value="GX16" x="30.48" y="91.44" smashed="yes"/>
 <element name="X7" library="con-subd" library_urn="urn:adsk.eagle:library:189" package="M09V" package3d_urn="urn:adsk.eagle:package:10298/1" value="" x="55.88" y="91.44" smashed="yes">
 <attribute name="MF" value="" x="44.958" y="71.628" size="1.778" layer="27" display="off"/>
@@
 <contactref element="X6" pad="X6"/>
 <contactref element="S1" pad="3"/>
-<wire x1="17.526" y1="89.154" x2="30.226" y2="91.44" width="0" layer="19" extent="1-1"/>
-<wire x1="16.002" y1="17.12" x2="17.526" y2="89.154" width="0" layer="19" extent="1-1"/>
+<via x="76.708" y="76.708" extent="1-16" drill="3.2"/>
+<via x="3.302" y="76.708" extent="1-16" drill="3.2"/>
+<via x="76.708" y="3.302" extent="1-16" drill="3.2"/>
+<via x="3.302" y="3.302" extent="1-16" drill="3.2"/>
+<wire x1="17.526" y1="89.154" x2="30.48" y2="91.44" width="0" layer="19" extent="1-1"/>
+<wire x1="3.302" y1="76.708" x2="17.526" y2="89.154" width="0" layer="19" extent="1-1"/>
 </signal>
 <signal name="3.3VREG">
@@
 <wire x1="65.4304" y1="53.0352" x2="58.6232" y2="92.8624" width="0" layer="19" extent="1-1"/>
 </signal>
-<signal name="GND2">
-<via x="76.708" y="76.708" extent="1-16" drill="3.2"/>
-</signal>
-<signal name="GND1">
-<via x="3.302" y="3.302" extent="1-16" drill="3.2"/>
-</signal>
-<signal name="GND3">
-<via x="3.302" y="76.708" extent="1-16" drill="3.2"/>
-</signal>
-<signal name="GND4" airwireshidden="yes">
-<via x="76.708" y="3.302" extent="1-16" drill="3.2"/>
-</signal>
 <signal name="GND5">
 <via x="76.2" y="91.44" extent="1-16" drill="3.2"/>
@@
 <contactref element="S1" pad="2"/>
 <contactref element="X6" pad="X1"/>
-<wire x1="14.986" y1="89.154" x2="26.416" y2="95.25" width="0" layer="19" extent="1-1"/>
+<wire x1="14.986" y1="89.154" x2="26.67" y2="95.25" width="0" layer="19" extent="1-1"/>
 </signal>
 <signal name="CZT_VIN">
